File: GridMaze/PCBs/maze_hub_1_1/maze_hub_1_1.brd (EAGLE design)
At the start: 154.2 x 39.5 mm, 29 parts, among them IC1 7805DT, IC2 TBD62083, IC3 PCA9517D, IC4 PCA9517D, IC5 MCP4541-104E/MS, IC6 OPA197

Commit message: Changes to 3x3 GridMaze hardware:
- Rather than seperate tall and short variants there is now a single intermediate height version of the maze.

- IR illumination is now provided by IR module PCBs which connect to the maze hub board using a Molex Micro-Fit cable and can be daisy chained.

- Reduced Poke IR beam current from 50mA to 40mA.
Parts:
- added J1: 430450210, Molex_430450210:MOLEX_430450210
- moved C1 20.1 mm to (12.3, 37.4), turned to 180 degrees
- moved C2 10.1 mm to (12.3, 24.7), turned to 180 degrees
- moved IC1 6.44 mm to (9.72, 31.1), turned to 90 degrees
- moved POW_CON 5.71 mm to (6.27, 6.67)
Connections:
- net +12V: now also J1.1
- net GND: now also J1.2
Routing:
- net +12V: track 359.5 -> 349.0 mm
- net RESET: track 99.4 -> 93.7 mm
- net GND: track 364.4 -> 360.5 mm
- net +5V: track 204.4 -> 206.7 mm
- net BNC-2: track 77.5 -> 75.8 mm
- net POW-4A: track 141.4 -> 142.9 mm
Other:
- board text added: "Licensed under the TAPR Open Hardware License (www.tapr.org/OHL) Copyright 2018-2025 Thomas Akam"
- board text added: "Maze_hub_1.1.1"
- board text removed: "Licensed under the TAPR Open Hardware License (www.tapr.org/OHL) Copyright 2018 Thomas Akam"
- board text removed: "Maze_hub_1_1"
