File: GridMaze/PCBs/maze_poke_1_0/maze_poke_1_0.brd (EAGLE design)
At the start: 20.5 x 69.2 mm, 16 parts

Commit message: Changes to 3x3 GridMaze hardware:
- Rather than seperate tall and short variants there is now a single intermediate height version of the maze.

- IR illumination is now provided by IR module PCBs which connect to the maze hub board using a Molex Micro-Fit cable and can be daisy chained.

- Reduced Poke IR beam current from 50mA to 40mA.
Parts:
- R1: value 82R -> 90R
Other:
- board text added: "Maze_poke_1.0.1"
- board text removed: "maze_poke_1_0"
Changed lines of the file:
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@@
 <wire x1="20.475" y1="0" x2="20.475" y2="69.18" width="0" layer="20"/>
 <wire x1="20.475" y1="69.18" x2="0" y2="69.18" width="0" layer="20"/>
-<text x="16.51" y="41.91" size="1.27" layer="21" rot="R180">maze_poke_1_0</text>
+<text x="16.51" y="41.91" size="1.27" layer="21" rot="R180">Maze_poke_1.0.1</text>
 <hole x="10.16" y="35.56" drill="2.8"/>
 <wire x1="0" y1="0" x2="0" y2="69.215" width="0" layer="20"/>
@@
 </autorouter>
 <elements>
-<element name="R1" library="resistor" package="R0805" value="82R" x="15.875" y="49.53" smashed="yes" rot="R90">
+<element name="R1" library="resistor" package="R0805" value="90R" x="15.875" y="49.53" smashed="yes" rot="R90">
 <attribute name="VALUE" x="18.2626" y="47.9044" size="0.9906" layer="27" ratio="10" rot="R90"/>
 </element>
